File: Hardware/Circuit/photogatePendulumKiCAD/20AL_Pendulum_Photogate.kicad_pcb (KiCad board)
At the start: 2 copper layers, 127 x 68.6 mm, 56 parts, among them Q1 2N3906, Q2 2N3904, Q3 2N3904, Q4 BPW40, Q5 2N3904, Q6 2N3904, Q7 2N3904, Q8 2N3904, SW2 SW_SPDT, U2 LM358

Commit message: Add instruction Pictures
Parts:
- moved SW2 2.59 mm to (95.0, 90.7)
Routing:
- net GND: track 289.1 -> 288.3 mm
Changed lines of the file:
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@@
 			(drillshape 0)
 			(scaleselection 1)
-			(outputdirectory "D:/photogate/")
+			(outputdirectory "../photogatePendulumGerber/")
 		)
 	)
@@
 	(footprint "User:SlideSwitch_SPDT"
 		(layer "F.Cu")
-		(at 95.504 88.138)
+		(at 94.996 90.678)
 		(descr "CuK miniature slide switch, OS series, SPDT, https://www.ckswitches.com/media/1428/os.pdf")
 		(tags "switch SPDT")
@@
 			(at 0.508 -2.921 0)
 			(layer "F.SilkS")
+			(hide yes)
 			(effects
 				(font
@@
 		(sheetfile "20AL_Pendulum_Photogate.kicad_sch")
 		(attr through_hole)
-		(fp_line
-			(start -6.731 -2.26)
-			(end 6.731 -2.26)
-			(stroke
-				(width 0.12)
-				(type solid)
-			)
-			(layer "F.SilkS")
-		)
-		(fp_line
-			(start -6.731 -1.95)
-			(end -6.731 -2.26)
-			(stroke
-				(width 0.12)
-				(type solid)
-			)
-			(layer "F.SilkS")
-		)
-		(fp_line
-			(start -6.731 2.26)
-			(end -6.731 1.877)
-			(stroke
-				(width 0.12)
-				(type solid)
-			)
-			(layer "F.SilkS")
-		)
-		(fp_line
-			(start -2.5 -2.96)
-			(end -2 -2.46)
-			(stroke
-				(width 0.12)
-				(type solid)
-			)
-			(layer "F.SilkS")
-		)
-		(fp_line
-			(start -2 -2.46)
-			(end -1.5 -2.96)
-			(stroke
-				(width 0.12)
-				(type solid)
-			)
-			(layer "F.SilkS")
-		)
-		(fp_line
-			(start -1.5 -2.96)
-			(end -2.5 -2.96)
-			(stroke
-				(width 0.12)
-				(type solid)
-			)
-			(layer "F.SilkS")
-		)
-		(fp_line
-			(start 6.731 -2.26)
-			(end 6.731 -1.95)
-			(stroke
-				(width 0.12)
-				(type solid)
-			)
-			(layer "F.SilkS")
-		)
-		(fp_line
-			(start 6.731 2.26)
-			(end -6.731 2.26)
-			(stroke
-				(width 0.12)
-				(type solid)
-			)
-			(layer "F.SilkS")
-		)
-		(fp_line
-			(start 6.731 2.26)
-			(end 6.731 1.95)
-			(stroke
-				(width 0.12)
-				(type solid)
-			)
-			(layer "F.SilkS")
-		)
 		(fp_rect
-			(start -7.11 -2.4)
-			(end 6.98 2.41)
+			(start -6.45 -2.8)
+			(end 6.45 3.1)
 			(stroke
-				(width 0.05)
+				(width 0.1)
 				(type default)
 			)
 			(fill no)
-			(layer "F.CrtYd")
+			(layer "F.SilkS")
 		)
 		(fp_line
@@
 			)
 		)
-		(pad "" thru_hole oval
-			(at -6.096 0)
-			(size 2.1844 3.556)
-			(drill 1.3716)
+		(pad "" thru_hole roundrect
+			(at -6.45 0)
+			(size 1.8288 2.54)
+			(drill oval 0.8128 2.54)
 			(layers "*.Cu" "*.Mask")
 			(remove_unused_layers no)
+			(roundrect_rratio 0.1367016623)
 		)
-		(pad "" thru_hole oval
-			(at 6.096 0)
-			(size 2.1844 3.556)
-			(drill 1.3716)
+		(pad "" thru_hole roundrect
+			(at 6.45 0)
+			(size 1.8288 2.54)
+			(drill oval 0.8128 2.54)
 			(layers "*.Cu" "*.Mask")
 			(remove_unused_layers no)
+			(roundrect_rratio 0.1367016623)
 		)
 		(pad "1" thru_hole roundrect
-			(at -2.794 0)
+			(at -3 0)
 			(size 2.032 2.54)
 			(drill 1.016)
@@
 		)
 		(pad "3" thru_hole oval
-			(at 2.794 0)
+			(at 3 0)
 			(size 2.032 2.54)
 			(drill 1.016)
@@
 		)
 	)
-	(gr_text "4n7"
+	(gr_text "1n"
 		(at 146.812 34.798 0)
 		(layer "User.3")
@@
 	)
 	(segment
-		(start 52.07 92.71)
-		(end 47.498 88.138)
+		(start 54.61 73.66)
+		(end 54.61 73.851413)
 		(width 0.508)
 		(layer "B.Cu")
@@
 	)
 	(segment
-		(start 121.92 92.71)
-		(end 116.84 92.71)
+		(start 110.49 92.71)
+		(end 110.109 93.091)
 		(width 0.508)
 		(layer "B.Cu")
@@
 	)
 	(segment
-		(start 96.774 84.836)
-		(end 98.298 86.36)
+		(start 35.023 58.928)
+		(end 34.29 58.195)
 		(width 0.508)
 		(layer "B.Cu")
@@
 	)
 	(segment
-		(start 41.91 71.882)
-		(end 38.262694 71.882)
+		(start 121.92 92.71)
+		(end 116.84 92.71)
 		(width 0.508)
 		(layer "B.Cu")
@@
 	)
 	(segment
-		(start 54.61 73.851413)
-		(end 52.6786 75.782813)
+		(start 38.262694 71.882)
+		(end 35.023 68.642306)
 		(width 0.508)
 		(layer "B.Cu")
@@
 	)
 	(segment
-		(start 98.552 92.71)
-		(end 52.07 92.71)
-		(width 0.508)
-		(layer "B.Cu")
-		(net 1)
-	)
-	(segment
-		(start 52.6786 79.3486)
-		(end 58.166 84.836)
-		(width 0.508)
-		(layer "B.Cu")
-		(net 1)
-	)
-	(segment
-		(start 54.61 73.66)
-		(end 54.61 73.851413)
-		(width 0.508)
-		(layer "B.Cu")
-		(net 1)
-	)
-	(segment
-		(start 129.286 92.67)
-		(end 132.831 92.67)
+		(start 94.869 85.217)
+		(end 97.996 88.344)
 		(width 0.508)
 		(layer "B.Cu")
@@
 	)
 	(segment
-		(start 58.166 84.836)
-		(end 96.774 84.836)
+		(start 129.286 92.67)
+		(end 132.831 92.67)
 		(width 0.508)
 		(layer "B.Cu")
@@
 	)
 	(segment
-		(start 38.262694 71.882)
-		(end 35.023 68.642306)
+		(start 97.996 93.043)
+		(end 98.044 93.091)
 		(width 0.508)
 		(layer "B.Cu")
@@
 	)
 	(segment
-		(start 110.49 92.71)
-		(end 98.552 92.71)
+		(start 97.996 90.678)
+		(end 97.996 93.043)
 		(width 0.508)
 		(layer "B.Cu")
@@
 	)
 	(segment
-		(start 125.262 92.67)
-		(end 125.222 92.71)
+		(start 35.023 68.642306)
+		(end 35.023 58.928)
 		(width 0.508)
 		(layer "B.Cu")
@@
 	)
 	(segment
-		(start 47.498 88.138)
-		(end 47.498 77.47)
+		(start 125.262 92.67)
+		(end 125.222 92.71)
 		(width 0.508)
 		(layer "B.Cu")
@@
 	)
 	(segment
-		(start 141.224 89.633)
-		(end 141.253 89.633)
+		(start 97.996 88.344)
+		(end 97.996 90.678)
 		(width 0.508)
 		(layer "B.Cu")
@@
 	)
 	(segment
-		(start 98.298 92.456)
-		(end 98.552 92.71)
+		(start 52.6786 79.3486)
+		(end 58.547 85.217)
 		(width 0.508)
 		(layer "B.Cu")
@@
 	)
 	(segment
-		(start 52.6786 75.782813)
-		(end 52.6786 79.3486)
+		(start 141.224 89.633)
+		(end 141.253 89.633)
 		(width 0.508)
 		(layer "B.Cu")
@@
 	)
 	(segment
-		(start 34.29 58.195)
-		(end 34.29 39.01)
+		(start 146.05 84.836)
+		(end 149.606 84.836)
 		(width 0.508)
 		(layer "B.Cu")
@@
 	)
 	(segment
-		(start 146.05 84.836)
-		(end 149.606 84.836)
+		(start 47.498 88.138)
+		(end 47.498 77.47)
 		(width 0.508)
 		(layer "B.Cu")
@@
 	)
 	(segment
-		(start 98.298 86.36)
-		(end 98.298 92.456)
+		(start 34.29 39.01)
+		(end 33.02 37.74)
 		(width 0.508)
 		(layer "B.Cu")
@@
 	)
 	(segment
+		(start 34.29 58.195)
+		(end 34.29 39.01)
+		(width 0.508)
+		(layer "B.Cu")
+		(net 1)
+	)
+	(segment
 		(start 151.13 41.881)
 		(end 151.159 41.91)
@@
 	)
 	(segment
+		(start 58.547 85.217)
+		(end 94.869 85.217)
+		(width 0.508)
+		(layer "B.Cu")
+		(net 1)
+	)
+	(segment
+		(start 54.61 73.851413)
+		(end 52.6786 75.782813)
+		(width 0.508)
+		(layer "B.Cu")
+		(net 1)
+	)
+	(segment
 		(start 127.254 92.67)
 		(end 125.262 92.67)
@@
 	)
 	(segment
-		(start 132.842 92.681)
-		(end 138.205 92.681)
+		(start 52.451 93.091)
+		(end 47.498 88.138)
 		(width 0.508)
 		(layer "B.Cu")
@@
 	)
 	(segment
-		(start 35.023 68.642306)
-		(end 35.023 58.928)
+		(start 41.91 71.882)
+		(end 38.262694 71.882)
 		(width 0.508)
 		(layer "B.Cu")
@@
 	)
 	(segment
-		(start 34.29 39.01)
-		(end 33.02 37.74)
+		(start 132.842 92.681)
+		(end 138.205 92.681)
 		(width 0.508)
 		(layer "B.Cu")
@@
 	)
 	(segment
+		(start 52.6786 75.782813)
+		(end 52.6786 79.3486)
+		(width 0.508)
+		(layer "B.Cu")
+		(net 1)
+	)
+	(segment
 		(start 151.13 63.558)
 		(end 151.13 71.882)
@@
 	)
 	(segment
-		(start 35.023 58.928)
-		(end 34.29 58.195)
+		(start 98.044 93.091)
+		(end 52.451 93.091)
+		(width 0.508)
+		(layer "B.Cu")
+		(net 1)
+	)
+	(segment
+		(start 110.109 93.091)
+		(end 98.044 93.091)
 		(width 0.508)
 		(layer "B.Cu")
@@
 	)
 	(segment
-		(start 75.994686 91.186)
-		(end 74.93 90.121314)
+		(start 74.93 87.678686)
+		(end 74.93 88.9)
 		(width 0.508)
 		(layer "B.Cu")
@@
 	)
 	(segment
-		(start 95.504 88.138)
-		(end 95.504 90.424)
+		(start 92.71 86.614)
+		(end 75.994686 86.614)
 		(width 0.508)
 		(layer "B.Cu")
@@
 	)
 	(segment
-		(start 94.742 91.186)
-		(end 75.994686 91.186)
+		(start 75.994686 86.614)
+		(end 74.93 87.678686)
 		(width 0.508)
 		(layer "B.Cu")
@@
 	)
 	(segment
-		(start 95.504 90.424)
-		(end 94.742 91.186)
+		(start 94.996 88.9)
+		(end 92.71 86.614)
 		(width 0.508)
 		(layer "B.Cu")
@@
 	)
 	(segment
-		(start 74.93 90.121314)
-		(end 74.93 88.9)
+		(start 94.996 90.678)
+		(end 94.996 88.9)
 		(width 0.508)
 		(layer "B.Cu")
